File: kicad/mini-speedo.kicad_pcb (KiCad board)
At the start: 2 copper layers, 3 parts, among them Q1 BC546, U1 LM2596T-5

Commit message: Schematics update, still not finished
Parts:
- added C1: 47uF, Capacitor_THT:CP_Radial_D6.3mm_P2.50mm, F.Cu at (148.6, 127.0)
- added C2: 33uF, Capacitor_THT:CP_Radial_D5.0mm_P2.50mm, F.Cu at (159.7, 112.7)
- added C3: 47uF, Capacitor_THT:CP_Radial_D6.3mm_P2.50mm, F.Cu at (210.5, 95.4)
- added C4: 33uF, Capacitor_THT:CP_Radial_D5.0mm_P2.50mm, F.Cu at (220.6, 89.5)
- added C5: 10uF, Capacitor_THT:CP_Radial_D5.0mm_P2.50mm, F.Cu at (226.6, 82.4)
- added C5: 10nF, Capacitor_THT:C_Rect_L4.0mm_W2.5mm_P2.50mm, F.Cu at (188.6, 145.1)
- added C6: 33nF, Capacitor_THT:C_Rect_L4.0mm_W2.5mm_P2.50mm, F.Cu at (232.7, 78.7)
- added D1: D_Schottky, Diode_THT:D_DO-35_SOD27_P7.62mm_Horizontal, F.Cu at (148.4, 104.1)
- added D10: 4.7V, Diode_SMD:D_MiniMELF_Handsoldering, F.Cu at (226.8, 74.9)
- added D11: 4.7V, Diode_SMD:D_MiniMELF_Handsoldering, F.Cu at (215.3, 84.4)
- added D12: 4.7V, Diode_SMD:D_MiniMELF_Handsoldering, F.Cu at (186.3, 134.5)
- added D13: 4.7V, Diode_SMD:D_MiniMELF_Handsoldering, F.Cu at (186.3, 137.7)
- added D2: 4.7V, Diode_SMD:D_MiniMELF_Handsoldering, F.Cu at (148.4, 107.7)
- added D3: 4.7V, Diode_SMD:D_MiniMELF_Handsoldering, F.Cu at (159.2, 104.1)
- added D4: 1N4148, Diode_THT:D_DO-35_SOD27_P7.62mm_Horizontal, F.Cu at (148.4, 111.2)
- added D5: 1N4148, Diode_THT:D_DO-35_SOD27_P7.62mm_Horizontal, F.Cu at (159.2, 107.7)
- added D6: 4.7V, Diode_SMD:D_MiniMELF_Handsoldering, B.Cu at (178.9, 104.4)
- added D7: 4.7V, Diode_SMD:D_MiniMELF_Handsoldering, F.Cu at (189.6, 104.4)
- added D8: 4.7V, Diode_SMD:D_MiniMELF_Handsoldering, F.Cu at (194.3, 80.0)
- added D9: 4.7V, Diode_SMD:D_MiniMELF_Handsoldering, F.Cu at (209.3, 89.7)
- added J1: Conn_01x06, Connector_Molex:Molex_Micro-Fit_3.0_43045-0600_2x03_P3.00mm_Horizontal, F.Cu at (243.8, 120.7)
- added J2: Conn_01x08, Connector_Molex:Molex_Micro-Fit_3.0_43045-0800_2x04_P3.00mm_Horizontal, F.Cu at (243.8, 137.2)
- added J3: Conn_01x10, Connector_Molex:Molex_Micro-Fit_3.0_43045-1000_2x05_P3.00mm_Horizontal, F.Cu at (243.8, 97.8)
- added J4: Conn_01x04, Connector_Molex:Molex_Micro-Fit_3.0_43045-0400_2x02_P3.00mm_Horizontal, F.Cu at (243.8, 156.2)
- added L1: 33uH, Ferrite_THT:LairdTech_28C0236-0JW-10, F.Cu at (167.6, 85.1)
- added Q2: BC546, Package_TO_SOT_THT:TO-92_Inline, F.Cu at (209.7, 102.5)
- added R1: 10k, Resistor_SMD:R_1206_3216Metric_Pad1.30x1.75mm_HandSolder, F.Cu at (157.8, 117.7)
- added R10: 100, Resistor_THT:R_Axial_DIN0207_L6.3mm_D2.5mm_P10.16mm_Horizontal, F.Cu at (217.2, 101.0)
- added R11: 470, Resistor_THT:R_Axial_DIN0207_L6.3mm_D2.5mm_P10.16mm_Horizontal, F.Cu at (224.6, 97.7)
- added R12: 15k, Resistor_SMD:R_1206_3216Metric_Pad1.30x1.75mm_HandSolder, F.Cu at (184.1, 141.0)
- added R13: 10k, Resistor_SMD:R_1206_3216Metric_Pad1.30x1.75mm_HandSolder, F.Cu at (184.1, 144.3)
- added R2: 10k, Resistor_SMD:R_1206_3216Metric_Pad1.30x1.75mm_HandSolder, F.Cu at (167.2, 112.9)
- added R3: 10k, Resistor_SMD:R_1206_3216Metric_Pad1.30x1.75mm_HandSolder, B.Cu at (203.2, 111.8)
- added R4: 10k, Resistor_SMD:R_1206_3216Metric_Pad1.30x1.75mm_HandSolder, F.Cu at (163.7, 117.7)
- added R5: 30k, Resistor_SMD:R_1206_3216Metric_Pad1.30x1.75mm_HandSolder, F.Cu at (218.7, 94.4)
- added R6: 10k, Resistor_SMD:R_1206_3216Metric_Pad1.30x1.75mm_HandSolder, F.Cu at (228.1, 87.3)
- added R7: 10k, Resistor_SMD:R_1206_3216Metric_Pad1.30x1.75mm_HandSolder, F.Cu at (218.7, 97.7)
- added R8: 10k, Resistor_SMD:R_1206_3216Metric_Pad1.30x1.75mm_HandSolder, F.Cu at (224.6, 94.4)
- added R9: 1k, Resistor_SMD:R_1206_3216Metric_Pad1.30x1.75mm_HandSolder, F.Cu at (228.1, 90.6)
- added U2: LM7810_TO220, Package_TO_SOT_THT:TO-220-3_Vertical, F.Cu at (161.3, 71.1)
- added U3: 74HC14, Package_SO:SO-14_3.9x8.65mm_P1.27mm, F.Cu at (200.7, 138.4)
- A1: value Arduino_Nano_v3.x -> Arduino
- moved U1 6.84 mm to (142.2, 74.9)
Connections:
- U1 pad 1: +BATT -> Net-(C1-Pad1)
Routing:
- net GND: track 17.7 -> 0.00 mm
