File: kicad/mini-speedo.sch (KiCad schematic (older format))
At the start: 15 parts, among them Q1 BC546, U1 LM2596T-5

Commit message: Further tests with kicad.
Parts:
- added J1a1: Conn stepper, symbol Connector:Conn_01x04_Female
- added J1b1: Conn stepper, symbol Connector:Conn_01x04_Male
- added J2a1: Conn display, symbol Connector:Conn_01x04_Female
- added J2b1: Conn display, symbol Connector:Conn_01x04_Male
- M1: renamed from M?; value Stepper_Motor_bipolar -> X27.168
- gave numbers to parts that had none: 1
Connections:
- net at M1.1: now also J1a1.1 (Pin_1)
- net at M1.2 (-): now also J1a1.2 (Pin_2)
- net at M1.3: now also J1a1.3 (Pin_3)
- net at M1.4: now also J1a1.4 (Pin_4)
Other:
- moved on the sheet: A1, C1, C2, D1, D2, D3, D4, L1, M1, Q1, R1, R2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

Commit message: KiCad changes, first prototype
Parts:
- removed R3: 10k, symbol Device:R
- added D?: 1N4148, Diode_THT:D_DO-35_SOD27_P7.62mm_Horizontal, symbol Diode:1N4148
Connections:
- net at A1.15 (D12): now also D?.1 (K)
- net at D3.1 (K), R2.1, U1.5 (~ON~/OFF): now also D?.2 (A)
Changed lines of the file:
@@
 Wire Wire Line
 	1200 1350 800  1350
-Connection ~ 2500 1150
-Wire Wire Line
-	2400 1150 2500 1150
-Wire Wire Line
-	2500 1350 2500 1150
 $Comp
 L Regulator_Switching:LM2596T-5 U1
@@
 	1    0    0    -1
 $EndComp
-$Comp
-L Device:R R3
-U 1 1 5F48AB45
-P 2500 1500
-F 0 "R3" H 2570 1546 50  0000 L CNN
-F 1 "10k" H 2570 1455 50  0000 L CNN
-F 2 "" V 2430 1500 50  0001 C CNN
-F 3 "~" H 2500 1500 50  0001 C CNN
-	1    2500 1500
-	1    0    0    -1
-$EndComp
-Wire Wire Line
-	2500 1650 2500 3450
 Wire Wire Line
 	5850 4550 5750 4550
@@
 Wire Wire Line
 	5950 950  5950 1150
-Wire Wire Line
-	2500 1150 2750 1150
 $Comp
 L Motor:Stepper_Motor_bipolar M1
@@
 Wire Wire Line
 	8550 1400 8500 1400
-Wire Bus Line
-	8400 1200 8400 1750
-Wire Bus Line
-	5100 1750 5100 2850
 Entry Wire Line
 	8500 1100 8400 1200
@@
 	-1   0    0    -1
 $EndComp
+Wire Wire Line
+	2400 1150 2500 1150
+$Comp
+L Diode:1N4148 D?
+U 1 1 5F9CBE2A
+P 2500 1550
+F 0 "D?" V 2546 1470 50  0000 R CNN
+F 1 "1N4148" V 2455 1470 50  0000 R CNN
+F 2 "Diode_THT:D_DO-35_SOD27_P7.62mm_Horizontal" H 2500 1375 50  0001 C CNN
+F 3 "https://assets.nexperia.com/documents/data-sheet/1N4148_1N4448.pdf" H 2500 1550 50  0001 C CNN
+	1    2500 1550
+	0    -1   -1   0
+$EndComp
+Wire Wire Line
+	2500 1400 2500 1150
+Connection ~ 2500 1150
+Wire Wire Line
+	2500 1150 2750 1150
+Wire Wire Line
+	2500 1700 2500 3450
+Wire Bus Line
+	8400 1200 8400 1750
+Wire Bus Line
+	5100 1750 5100 2850
 $EndSCHEMATC

Commit message: Schematics update, still not finished
Parts:
- removed J1a1: Conn stepper, symbol Connector:Conn_01x04_Female
- removed J1b1: Conn stepper, symbol Connector:Conn_01x04_Male
- removed J2a1: Conn display, symbol Connector:Conn_01x04_Female
- removed J2b1: Conn display, symbol Connector:Conn_01x04_Male
- added C3: 47uF, Capacitor_THT:CP_Radial_D6.3mm_P2.50mm, symbol Device:CP
- added C4: 33uF, Capacitor_THT:CP_Radial_D5.0mm_P2.50mm, symbol Device:CP
- added C5: 10nF, Capacitor_THT:C_Rect_L4.0mm_W2.5mm_P2.50mm, symbol Device:C
- added C6: 33nF, Capacitor_THT:C_Rect_L4.0mm_W2.5mm_P2.50mm, symbol Device:C
- added D10, D11, D12, D13, D6, D7, D8, D9: 4.7V, Diode_SMD:D_MiniMELF_Handsoldering, symbol Device:D_Zener
- added J1: Conn_01x06, Connector_Molex:Molex_Micro-Fit_3.0_43045-0600_2x03_P3.00mm_Horizontal, symbol Connector_Generic:Conn_01x06
- added J2: Conn_01x08, Connector_Molex:Molex_Micro-Fit_3.0_43045-0800_2x04_P3.00mm_Horizontal, symbol Connector_Generic:Conn_01x08
- added J3: Conn_01x10, Connector_Molex:Molex_Micro-Fit_3.0_43045-1000_2x05_P3.00mm_Horizontal, symbol Connector_Generic:Conn_01x10
- added J4: Conn_01x04, Connector_Molex:Molex_Micro-Fit_3.0_43045-0400_2x02_P3.00mm_Horizontal, symbol Connector_Generic:Conn_01x04
- added Q2: BC546, Package_TO_SOT_THT:TO-92_Inline, symbol Transistor_BJT:BC546
- added R10: 100, Resistor_THT:R_Axial_DIN0207_L6.3mm_D2.5mm_P10.16mm_Horizontal, symbol Device:R
- added R11: 470, Resistor_THT:R_Axial_DIN0207_L6.3mm_D2.5mm_P10.16mm_Horizontal, symbol Device:R
- added R12: 15k, Resistor_SMD:R_1206_3216Metric_Pad1.30x1.75mm_HandSolder, symbol Device:R
- added R13, R3, R6, R7, R8: 10k, Resistor_SMD:R_1206_3216Metric_Pad1.30x1.75mm_HandSolder, symbol Device:R
- added R5: 30k, Resistor_SMD:R_1206_3216Metric_Pad1.30x1.75mm_HandSolder, symbol Device:R
- added R9: 1k, Resistor_SMD:R_1206_3216Metric_Pad1.30x1.75mm_HandSolder, symbol Device:R
- added U2: LM7810_TO220, Package_TO_SOT_THT:TO-220-3_Vertical, symbol Regulator_Linear:LM7810_TO220
- added U3: 74HC14, Package_SO:SO-14_3.9x8.65mm_P1.27mm, symbol 74xx:74HC14
- A1: value Arduino_Nano_v3.x -> Arduino
- C1: footprint (none) -> Capacitor_THT:CP_Radial_D6.3mm_P2.50mm
- C2: footprint (none) -> Capacitor_THT:CP_Radial_D5.0mm_P2.50mm
- D1: footprint (none) -> Diode_THT:D_DO-35_SOD27_P7.62mm_Horizontal
- D2, D3: footprint (none) -> Diode_SMD:D_MiniMELF_Handsoldering
- D4: value D -> 1N4148; footprint (none) -> Diode_THT:D_DO-35_SOD27_P7.62mm_Horizontal
- L1: footprint (none) -> Ferrite_THT:LairdTech_28C0236-0JW-10
- R1, R2, R4: footprint (none) -> Resistor_SMD:R_1206_3216Metric_Pad1.30x1.75mm_HandSolder
- gave numbers to parts that had none: 1
Connections:
- net GND: now also C3.2, C4.2, C5.2, C6.2, D10.2 (A), D11.2 (A), D13.2 (A), D6.2 (A), D7.2 (A), D8.2 (A), D9.2 (A), J1.6 (Pin_6), J2.8 (Pin_8), J3.2 (Pin_2), J4.4 (Pin_4), Q2.3 (E), R13.1, R6.1, R7.1, U2.2 (GND), U3.7 (GND)
- net at A1.10 (D7): now also J2.4 (Pin_4)
- net at A1.11 (D8): no longer D4.2 (A)
- net at A1.13 (D10): now also D4.2 (A)
- net at A1.16 (D13): now also R3.1
- net at A1.19 (A0): now also J3.3 (Pin_3)
- net at A1.20 (A1): now also D11.1 (K), J3.5 (Pin_5), R11.1
- net at A1.21 (A2): now also D10.1 (K), J3.6 (Pin_6), R10.1
- net at A1.22 (A3): now also D9.1 (K), J3.7 (Pin_7)
- net at A1.23 (A4): now also J2.6 (Pin_6)
- net at A1.24 (A5): now also J2.7 (Pin_7)
- net at A1.25 (A6): now also C6.1, D7.1 (K), R7.2, R8.1
- net at A1.26 (A7): now also D6.1 (K), R5.1, R6.2
- net at A1.27 (+5V), C2.1, L1.1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: now also D12.1 (K), J2.5 (Pin_5), J3.1 (Pin_1), R10.2, R11.2, U3.14 (VCC)
- net at A1.5 (D2): now also U3.4
- net at A1.6 (D3): now also U3.2
- net at A1.7 (D4): now also J2.1 (Pin_1)
- net at A1.8 (D5): now also J2.2 (Pin_2)
- net at A1.9 (D6): now also J2.3 (Pin_3)
- net at D4.1 (K): now also J1.4 (Pin_4)
- net +BATT: no longer names the net of C1.1, U1.1 (VIN)
- net +BATT: now also J1.1 (Pin_1)
- net VDC: no longer names the net of R1.2, R4.2
- net VDC: now also C3.1, J1.2 (Pin_2), J4.2 (Pin_2), R5.2, U2.1 (VI)
- new net: J1.5 (Pin_5), Q2.1 (C)
- new net: Q2.2 (B), R3.2
- new net: C4.1, J1.3 (Pin_3), U2.3 (VO)
- new net: J4.1 (Pin_1), R12.2
- new net: J4.3 (Pin_3), R9.2
- new net: J3.4 (Pin_4), R8.2
- new net: D8.1 (K), R9.1, U3.3
- new net: C5.1, D12.2 (A), D13.1 (K), R12.1, R13.2, U3.1
Other:
- note added: "max3232"
- moved on the sheet: A1, D2, D3, D4, D5, R4
